File: rev0/aux_port.kicad_sch (KiCad schematic)
At the start: 27 parts, among them IC1 ECP5-BGA256, U11 USB3343-CP, U12 FUSB302BMPX, U14 DPO2036

Commit message: hardware: component placement
Connections:
- net AUX_CC1: now also C52.1
- net AUX_CC1S: no longer C52.1
- net AUX_CC2: now also C53.1
- net AUX_CC2S: no longer C53.1
Other:
- moved on the sheet: C52, C53
Changed lines of the file:
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@@
   (junction (at 168.91 27.94) (diameter 0) (color 0 0 0 0)
   )
+  (junction (at 241.3 52.705) (diameter 0) (color 0 0 0 0)
+  )
+  (junction (at 251.46 55.245) (diameter 0) (color 0 0 0 0)
+  )
   (junction (at 118.11 173.99) (diameter 0) (color 0 0 0 0)
   )
@@
   (junction (at 213.36 66.675) (diameter 0) (color 0 0 0 0)
   )
-  (junction (at 139.7 70.485) (diameter 0) (color 0 0 0 0)
-  )
-  (junction (at 149.86 60.325) (diameter 0) (color 0 0 0 0)
+  (junction (at 241.3 65.405) (diameter 0) (color 0 0 0 0)
   )
   (junction (at 262.89 33.02) (diameter 0) (color 0 0 0 0)
-  )
-  (junction (at 139.7 57.785) (diameter 0) (color 0 0 0 0)
   )
   (junction (at 262.89 22.86) (diameter 0) (color 0 0 0 0)
@@
     (stroke (width 0) (type default) (color 0 0 0 0))
   )
-  (wire (pts (xy 139.7 57.785) (xy 201.93 57.785))
+  (wire (pts (xy 133.35 57.785) (xy 201.93 57.785))
     (stroke (width 0) (type default) (color 0 0 0 0))
   )
@@
     (stroke (width 0) (type default) (color 0 0 0 0))
   )
-  (wire (pts (xy 224.79 55.245) (xy 227.33 55.245))
+  (wire (pts (xy 224.79 55.245) (xy 251.46 55.245))
     (stroke (width 0) (type default) (color 0 0 0 0))
   )
@@
     (stroke (width 0) (type default) (color 0 0 0 0))
   )
-  (wire (pts (xy 149.86 60.325) (xy 133.35 60.325))
-    (stroke (width 0) (type default) (color 0 0 0 0))
-  )
   (wire (pts (xy 232.41 104.14) (xy 227.33 104.14))
     (stroke (width 0) (type default) (color 0 0 0 0))
@@
     (stroke (width 0) (type default) (color 0 0 0 0))
   )
-  (wire (pts (xy 139.7 70.485) (xy 149.86 70.485))
+  (wire (pts (xy 241.3 65.405) (xy 251.46 65.405))
     (stroke (width 0) (type default) (color 0 0 0 0))
   )
@@
     (stroke (width 0) (type default) (color 0 0 0 0))
   )
-  (wire (pts (xy 149.86 61.595) (xy 149.86 60.325))
+  (wire (pts (xy 251.46 56.515) (xy 251.46 55.245))
     (stroke (width 0) (type default) (color 0 0 0 0))
   )
@@
     (stroke (width 0) (type default) (color 0 0 0 0))
   )
-  (wire (pts (xy 149.86 70.485) (xy 149.86 69.215))
+  (wire (pts (xy 251.46 65.405) (xy 251.46 64.135))
     (stroke (width 0) (type default) (color 0 0 0 0))
   )
@@
     (stroke (width 0) (type default) (color 0 0 0 0))
   )
+  (wire (pts (xy 251.46 55.245) (xy 254 55.245))
+    (stroke (width 0) (type default) (color 0 0 0 0))
+  )
   (bus (pts (xy 148.59 128.27) (xy 148.59 130.81))
     (stroke (width 0) (type default) (color 0 0 0 0))
@@
     (stroke (width 0) (type default) (color 0 0 0 0))
   )
-  (wire (pts (xy 149.86 60.325) (xy 201.93 60.325))
+  (wire (pts (xy 133.35 60.325) (xy 201.93 60.325))
     (stroke (width 0) (type default) (color 0 0 0 0))
   )
@@
     (stroke (width 0) (type default) (color 0 0 0 0))
   )
-  (wire (pts (xy 139.7 61.595) (xy 139.7 57.785))
+  (wire (pts (xy 241.3 56.515) (xy 241.3 52.705))
     (stroke (width 0) (type default) (color 0 0 0 0))
   )
@@
     (stroke (width 0) (type default) (color 0 0 0 0))
   )
-  (wire (pts (xy 139.7 69.215) (xy 139.7 70.485))
-    (stroke (width 0) (type default) (color 0 0 0 0))
-  )
-  (wire (pts (xy 224.79 52.705) (xy 227.33 52.705))
+  (wire (pts (xy 241.3 64.135) (xy 241.3 65.405))
+    (stroke (width 0) (type default) (color 0 0 0 0))
+  )
+  (wire (pts (xy 224.79 52.705) (xy 241.3 52.705))
     (stroke (width 0) (type default) (color 0 0 0 0))
   )
@@
     (stroke (width 0) (type default) (color 0 0 0 0))
   )
-  (wire (pts (xy 139.7 70.485) (xy 139.7 71.755))
+  (wire (pts (xy 241.3 65.405) (xy 241.3 66.675))
     (stroke (width 0) (type default) (color 0 0 0 0))
   )
@@
     (stroke (width 0) (type default) (color 0 0 0 0))
   )
-  (wire (pts (xy 133.35 57.785) (xy 139.7 57.785))
+  (wire (pts (xy 241.3 52.705) (xy 254 52.705))
     (stroke (width 0) (type default) (color 0 0 0 0))
   )
@@
     (effects (font (size 1.27 1.27)) (justify left))
   )
-  (hierarchical_label "AUX_CC1" (shape bidirectional) (at 227.33 52.705 0)
+  (hierarchical_label "AUX_CC1" (shape bidirectional) (at 254 52.705 0)
     (effects (font (size 1.27 1.27)) (justify left))
   )
-  (hierarchical_label "AUX_CC2" (shape bidirectional) (at 227.33 55.245 0)
+  (hierarchical_label "AUX_CC2" (shape bidirectional) (at 254 55.245 0)
     (effects (font (size 1.27 1.27)) (justify left))
   )
@@
     (pin "2")
   )
-  (symbol (lib_id "power:GND") (at 139.7 71.755 0) (mirror y) (unit 1)
+  (symbol (lib_id "power:GND") (at 241.3 66.675 0) (mirror y) (unit 1)
     (in_bom yes) (on_board yes) (fields_autoplaced)
-    (property "Reference" "#PWR06" (id 0) (at 139.7 78.105 0)
-      (effects (font (size 1.27 1.27)) hide)
-    )
-    (property "Value" "GND" (id 1) (at 139.7 76.1984 0))
-    (property "Footprint" "" (id 2) (at 139.7 71.755 0)
-      (effects (font (size 1.27 1.27)) hide)
-    )
-    (property "Datasheet" "" (id 3) (at 139.7 71.755 0)
+    (property "Reference" "#PWR06" (id 0) (at 241.3 73.025 0)
+      (effects (font (size 1.27 1.27)) hide)
+    )
+    (property "Value" "GND" (id 1) (at 241.3 71.1184 0))
+    (property "Footprint" "" (id 2) (at 241.3 66.675 0)
+      (effects (font (size 1.27 1.27)) hide)
+    )
+    (property "Datasheet" "" (id 3) (at 241.3 66.675 0)
       (effects (font (size 1.27 1.27)) hide)
     )
@@
     (pin "2")
   )
-  (symbol (lib_id "Device:C") (at 139.7 65.405 0) (unit 1)
-    (in_bom yes) (on_board yes)
-    (property "Reference" "C52" (id 0) (at 140.97 62.865 0)
-      (effects (font (size 1.27 1.27)) (justify left))
-    )
-    (property "Value" "390pF" (id 1) (at 140.97 67.945 0)
-      (effects (font (size 1.27 1.27)) (justify left))
-    )
-    (property "Footprint" "Capacitor_SMD:C_0402_1005Metric" (id 2) (at 140.6652 69.215 0)
-      (effects (font (size 1.27 1.27)) hide)
-    )
-    (property "Datasheet" "~" (id 3) (at 139.7 65.405 0)
-      (effects (font (size 1.27 1.27)) hide)
-    )
-    (property "Part Number" "GENERIC-CAP-0402-390pF" (id 4) (at 139.7 65.405 0)
-      (effects (font (size 1.27 1.27)) hide)
-    )
-    (property "Substitution" "any equivalent" (id 5) (at 139.7 65.405 0)
+  (symbol (lib_id "Device:C") (at 241.3 60.325 0) (unit 1)
+    (in_bom yes) (on_board yes)
+    (property "Reference" "C52" (id 0) (at 242.57 57.785 0)
+      (effects (font (size 1.27 1.27)) (justify left))
+    )
+    (property "Value" "390pF" (id 1) (at 242.57 62.865 0)
+      (effects (font (size 1.27 1.27)) (justify left))
+    )
+    (property "Footprint" "Capacitor_SMD:C_0402_1005Metric" (id 2) (at 242.2652 64.135 0)
+      (effects (font (size 1.27 1.27)) hide)
+    )
+    (property "Datasheet" "~" (id 3) (at 241.3 60.325 0)
+      (effects (font (size 1.27 1.27)) hide)
+    )
+    (property "Part Number" "GENERIC-CAP-0402-390pF" (id 4) (at 241.3 60.325 0)
+      (effects (font (size 1.27 1.27)) hide)
+    )
+    (property "Substitution" "any equivalent" (id 5) (at 241.3 60.325 0)
       (effects (font (size 1.27 1.27)) hide)
     )
@@
     (pin "9")
   )
-  (symbol (lib_id "Device:C") (at 149.86 65.405 0) (unit 1)
-    (in_bom yes) (on_board yes)
-    (property "Reference" "C53" (id 0) (at 151.13 62.865 0)
-      (effects (font (size 1.27 1.27)) (justify left))
-    )
-    (property "Value" "390pF" (id 1) (at 151.13 67.945 0)
-      (effects (font (size 1.27 1.27)) (justify left))
-    )
-    (property "Footprint" "Capacitor_SMD:C_0402_1005Metric" (id 2) (at 150.8252 69.215 0)
-      (effects (font (size 1.27 1.27)) hide)
-    )
-    (property "Datasheet" "~" (id 3) (at 149.86 65.405 0)
-      (effects (font (size 1.27 1.27)) hide)
-    )
-    (property "Part Number" "GENERIC-CAP-0402-390pF" (id 4) (at 149.86 65.405 0)
-      (effects (font (size 1.27 1.27)) hide)
-    )
-    (property "Substitution" "any equivalent" (id 5) (at 149.86 65.405 0)
-      (effects (font (size 1.27 1.27)) hide)
-    )
+  (symbol (lib_id "Device:C") (at 251.46 60.325 0) (unit 1)
+    (in_bom yes) (on_board yes)
+    (property "Reference" "C53" (id 0) (at 252.73 57.785 0)
+      (effects (font (size 1.27 1.27)) (justify left))
+    )
+    (property "Value" "390pF" (id 1) (at 252.73 62.865 0)
+      (effects (font (size 1.27 1.27)) (justify left))
+    )
+    (property "Footprint" "Capacitor_SMD:C_0402_1005Metric" (id 2) (at 252.4252 64.135 0)
+      (effects (font (size 1.27 1.27)) hide)
+    )
+    (property "Datasheet" "~" (id 3) (at 251.46 60.325 0)
+      (effects (font (size 1.27 1.27)) hide)
+    )
+    (property "Part Number" "GENERIC-CAP-0402-390pF" (id 4) (at 251.46 60.325 0)
+      (effects (font (size 1.27 1.27)) hide)
+    )
+    (property "Substitution" "any equivalent" (id 5) (at 251.46 60.325 0)
+      (effects (font (size 1.27 1.27)) hide)
+    )
